File: hardware/main_board/video_switching.kicad_sch (KiCad schematic)
At the start: 33 parts, among them SW1 rgb/ypbpr, SW2 rgb/ypbpr, SW3 rgb/ypbpr, SW4 rgb/ypbpr, SW5 rgb/ypbpr, SW6 rgb/ypbpr, SW7 rgb/ypbpr, SW8 rgb/ypbpr, U10 SN74CBT3244CPW, U11 SN74CBT3244CPW, U12 SN74CBT3244CPW, U13 SN74CBT3244CPW, U14 74HC238, U15 74HC238, U3 SN74CBT3244CPW, U4 SN74CBT3244CPW, U5 74HC138, U6 74HC04, U7 SN74CBT3244CPW, U8 SN74CBT3244CPW, U9 SN74CBT3244CPW

Commit message: #1: Removed audio biasing circuitry as it's apparently unnecessary.
Connections:
- net AudioLIn0Biased renamed AudioLIn0
- net AudioLIn1Biased renamed AudioLIn1
- net AudioLIn2Biased renamed AudioLIn2
- net AudioLIn3Biased renamed AudioLIn3
- net AudioLIn4Biased renamed AudioLIn4
- net AudioLIn5Biased renamed AudioLIn5
- net AudioLIn6Biased renamed AudioLIn6
- net AudioLIn7Biased renamed AudioLIn7
- net AudioLOutBiased renamed AudioLOut
- net AudioRIn0Biased renamed AudioRIn0
- net AudioRIn1Biased renamed AudioRIn1
- net AudioRIn2Biased renamed AudioRIn2
- net AudioRIn3Biased renamed AudioRIn3
- net AudioRIn4Biased renamed AudioRIn4
- net AudioRIn5Biased renamed AudioRIn5
- net AudioRIn6Biased renamed AudioRIn6
- net AudioRIn7Biased renamed AudioRIn7
- net AudioROutBiased renamed AudioROut
Other:
- removed sheet audio biasing
- moved on the sheet: SW1, SW2, SW3, SW4, SW5, SW6, SW7, SW8
