File: hardware/main_board/main_board.kicad_pcb (KiCad board)
At the start: 4 copper layers, 225.9 x 135 mm, 89 parts, among them J1 +5v in, J10 uart, J11 input 4, J12 input 5, J14 +5v in/out, J16 input 6, J17 input 7, J19 rgb output, J20 ypbpr output, J3 input 0, J4 input 1, J5 icsp, J7 input 2, J8 input 3, SW1 rgb/ypbpr, SW10 prev, SW11 next, SW12 csync/rgbs, SW13 csync/rgbs, SW14 csync/rgbs, SW15 csync/rgbs, SW16 csync/rgbs, SW17 csync/rgbs, SW18 csync/rgbs, SW19 csync/rgbs, SW2 rgb/ypbpr, SW20 csync/rgbs, SW3 rgb/ypbpr, SW4 rgb/ypbpr, SW5 rgb/ypbpr, SW6 rgb/ypbpr, SW7 rgb/ypbpr, SW8 rgb/ypbpr, U1 ATmega328PB-A, U10 SN74CBT3244CPW, U11 SN74CBT3244CPW, U12 SN74CBT3244CPW, U13 SN74CBT3244CPW, U14 74HC238, U15 74HC238, U3 SN74CBT3244CPW, U4 SN74CBT3244CPW, U5 74HC138, U6 74HC04, U7 SN74CBT3244CPW, U8 SN74CBT3244CPW, U9 SN74CBT3244CPW

Commit message: #5: Fixed botched dimensions again...it's only by 0.1mm in the x direction and I can't be bothered redoing the render a 3rd time.
Parts:
- moved H4 3.19 mm to (252.4, 145.3)
- moved H2 3.19 mm to (252.4, 30.3)
- moved J14 3.14 mm to (256.1, 126.3)
- moved C1 3.14 mm to (174.0, 67.7)
- moved C10 3.14 mm to (185.8, 135.1)
- moved C11 3.14 mm to (167.4, 135.1)
- moved C12 3.14 mm to (149.0, 135.1)
- moved C13 3.14 mm to (130.6, 135.1)
- moved C14 3.14 mm to (113.2, 134.2)
- moved C15 3.14 mm to (94.0, 135.1)
- moved C18 3.14 mm to (66.4, 129.3)
- moved C19 3.14 mm to (129.6, 48.3)
- moved C2 3.14 mm to (174.4, 70.1)
- moved C3 3.14 mm to (47.0, 132.3)
- moved C4 3.14 mm to (45.2, 131.0)
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Other:
- board size 225.9 x 135 mm -> 226 x 135 mm
