File: hardware/led_board/led_board.kicad_sch (KiCad schematic)
At the start: 56 parts, among them J1 icsp, J10 rgb 2, J11 rgb 7, J12 rgb 5, J2 +5v out, J3 uart, J4 rgb 0, J5 rgb 3, J6 +12v 3a in, J7 rgb 4, J8 rgb 6, J9 rgb 1, Q1 IRF540N, Q10 IRF540N, Q11 IRF540N, Q12 IRF540N, Q13 IRF540N, Q14 IRF540N, Q15 IRF540N, Q16 IRF540N, Q17 IRF540N, Q18 IRF540N, Q19 IRF540N, Q2 IRF540N, Q20 IRF540N, Q21 IRF540N, Q22 IRF540N, Q23 IRF540N, Q24 IRF540N, Q25 IRF540N, Q26 IRF540N, Q27 IRF540N, Q28 IRF540N, Q29 IRF540N, Q3 IRF540N, Q30 IRF540N, Q31 IRF540N, Q32 IRF540N, Q4 IRF540N, Q5 IRF540N, Q6 IRF540N, Q7 IRF540N, Q8 IRF540N, Q9 IRF540N, SW1 on/off, U1 ATmega328PB-A, U2 L7805

Commit message: #5: We have a completed LED board! 🎉
Parts:
- added H1, H2, H3, H4: ground, MountingHole:MountingHole_4.3mm_M4_ISO14580_Pad, symbol Mechanical:MountingHole_Pad
Connections:
- net GND: now also H1.1, H2.1, H3.1, H4.1
Other:
- note added: "mounting holes"
